Commit message: Update Week 7 ground gimbal robot package

File: src/ground_gimbal_robot/urdf/ground_gimbal_robot.xacro (robot description, xacro)
@@ -478,4 +478,14 @@
     <origin xyz="-0.17 0 ${caster_radius - wheel_radius}" rpy="0 0 0"/>
   </joint>
+  <gazebo reference="front_caster_link">
+    <material>Gazebo/Grey</material>
+    <mu1>0.02</mu1>
+    <mu2>0.02</mu2>
+  </gazebo>
+  <gazebo reference="rear_caster_link">
+    <material>Gazebo/Grey</material>
+    <mu1>0.02</mu1>
+    <mu2>0.02</mu2>
+  </gazebo>
   <gazebo reference="base_link">
     <material>Gazebo/DarkGrey</material>
@@ -559,7 +569,6 @@
     <plugin name="ground_gimbal_diff_drive" filename="libgazebo_ros_diff_drive.so">
       <ros>
-        <namespace>/</namespace>
-        <remapping>cmd_vel:=cmd_vel</remapping>
-        <remapping>odom:=odom</remapping>
+        <remapping>cmd_vel:=/cmd_vel</remapping>
+        <remapping>odom:=/odom</remapping>
       </ros>
       <left_joint>left_wheel_joint</left_joint>
@@ -569,6 +578,6 @@
       <max_wheel_torque>20.0</max_wheel_torque>
       <max_wheel_acceleration>4.0</max_wheel_acceleration>
-      <command_topic>cmd_vel</command_topic>
-      <odometry_topic>odom</odometry_topic>
+      <command_topic>/cmd_vel</command_topic>
+      <odometry_topic>/odom</odometry_topic>
       <odometry_frame>odom</odometry_frame>
       <robot_base_frame>base_footprint</robot_base_frame>

Commit message: Add final YOLO gimbal robot demo

File: src/ground_gimbal_robot/urdf/ground_gimbal_robot.xacro (robot description, xacro)
@@ -208,4 +208,27 @@
     <origin xyz="0.08 0 ${base_height}" rpy="0 0 0"/>
   </joint>
+  <link name="lidar_link">
+    <visual>
+      <origin xyz="0 0 0.018" rpy="0 0 0"/>
+      <geometry>
+        <cylinder radius="0.045" length="0.036"/>
+      </geometry>
+      <material name="lidar_black">
+        <color rgba="0.015 0.018 0.02 1.0"/>
+      </material>
+    </visual>
+    <collision>
+      <origin xyz="0 0 0.018" rpy="0 0 0"/>
+      <geometry>
+        <cylinder radius="0.045" length="0.036"/>
+      </geometry>
+    </collision>
+    <xacro:cylinder_inertia mass="0.12" radius="0.045" length="0.036" axis="z"/>
+  </link>
+  <joint name="lidar_joint" type="fixed">
+    <parent link="base_link"/>
+    <child link="lidar_link"/>
+    <origin xyz="0.34 0 ${base_height + 0.10}" rpy="0 0 0"/>
+  </joint>
   <link name="gimbal_pan_link">
     <visual>
@@ -250,10 +273,10 @@
   </xacro:if>
   <xacro:unless value="$(arg gazebo_static_gimbal)">
-    <joint name="gimbal_pan_joint" type="revolute">
+    <joint name="gimbal_pan_joint" type="continuous">
       <parent link="gimbal_mount_link"/>
       <child link="gimbal_pan_link"/>
       <origin xyz="0 0 ${mount_height + 0.036}" rpy="0 0 0"/>
       <axis xyz="0 0 1"/>
-      <limit lower="-3.14159" upper="3.14159" effort="4.0" velocity="2.5"/>
+      <limit effort="4.0" velocity="2.5"/>
       <dynamics damping="0.15" friction="0.02"/>
     </joint>
@@ -556,4 +579,41 @@
     </sensor>
   </gazebo>
+  <gazebo reference="lidar_link">
+    <material>Gazebo/Black</material>
+    <sensor name="front_lidar" type="ray">
+      <pose>0 0 0.025 0 0 0</pose>
+      <always_on>true</always_on>
+      <visualize>true</visualize>
+      <update_rate>10</update_rate>
+      <ray>
+        <scan>
+          <horizontal>
+            <samples>271</samples>
+            <resolution>1</resolution>
+            <min_angle>-2.35619</min_angle>
+            <max_angle>2.35619</max_angle>
+          </horizontal>
+        </scan>
+        <range>
+          <min>0.22</min>
+          <max>8.0</max>
+          <resolution>0.01</resolution>
+        </range>
+        <noise>
+          <type>gaussian</type>
+          <mean>0.0</mean>
+          <stddev>0.01</stddev>
+        </noise>
+      </ray>
+      <plugin name="front_lidar_controller" filename="libgazebo_ros_ray_sensor.so">
+        <ros>
+          <namespace>/</namespace>
+          <remapping>~/out:=scan</remapping>
+        </ros>
+        <output_type>sensor_msgs/LaserScan</output_type>
+        <frame_name>lidar_link</frame_name>
+      </plugin>
+    </sensor>
+  </gazebo>
   <gazebo reference="left_wheel_link">
     <material>Gazebo/Black</material>
